File: Schematic/MascotDesign/Amplifier_Circuit.kicad_sch (KiCad schematic)
At the start: 32 parts, among them J10 AudioJack4, J5 Audio in, J6 Audio in, J8 Potentiometer, J9 Speaker 8R, U3 TPA3116D2DAD

Commit message: Merge branch 'main' of https://github.com/DrGlaucous/mascot-head-sr-design
Connections:
- net at C2.2, J5.2 (Pin_2), J6.2 (Pin_2): now also J10.T; no longer J10.S
- net at C1.1, J5.1 (Pin_1), J6.1 (Pin_1): now also J10.S; no longer J10.T
Changed lines of the file:
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@@
-	)
-	(junction
-		(at 44.45 64.77)
-		(diameter 0)
-		(color 0 0 0 0)
 	)
 	(junction
@@
 	)
 	(junction
+		(at 44.45 57.15)
+		(diameter 0)
+		(color 0 0 0 0)
+	)
+	(junction
 		(at 176.53 76.2)
 		(diameter 0)
@@
 	)
 	(junction
-		(at 57.15 57.15)
+		(at 57.15 64.77)
 		(diameter 0)
 		(color 0 0 0 0)
@@
 	(wire
 		(pts
+			(xy 38.1 57.15) (xy 44.45 57.15)
+		)
+		(stroke
+			(width 0)
+			(type default)
+		)
+	)
+	(wire
+		(pts
 			(xy 44.45 38.1) (xy 44.45 50.8)
 		)
@@
 	(wire
 		(pts
-			(xy 44.45 50.8) (xy 44.45 64.77)
-		)
-		(stroke
-			(width 0)
-			(type default)
-		)
-	)
-	(wire
-		(pts
 			(xy 175.26 73.66) (xy 176.53 73.66)
 		)
@@
 	(wire
 		(pts
+			(xy 44.45 57.15) (xy 44.45 73.66)
+		)
+		(stroke
+			(width 0)
+			(type default)
+		)
+	)
+	(wire
+		(pts
 			(xy 176.53 76.2) (xy 176.53 78.74)
 		)
@@
 	(wire
 		(pts
-			(xy 44.45 64.77) (xy 44.45 73.66)
+			(xy 44.45 50.8) (xy 44.45 57.15)
 		)
 		(stroke
@@
 	(wire
 		(pts
-			(xy 38.1 64.77) (xy 44.45 64.77)
-		)
-		(stroke
-			(width 0)
-			(type default)
-		)
-	)
-	(wire
-		(pts
 			(xy 38.1 48.26) (xy 57.15 48.26)
 		)
@@
 	(wire
 		(pts
-			(xy 38.1 57.15) (xy 57.15 57.15)
-		)
-		(stroke
-			(width 0)
-			(type default)
-		)
-	)
-	(wire
-		(pts
 			(xy 38.1 86.36) (xy 90.17 86.36)
 		)
@@
 	(wire
 		(pts
-			(xy 57.15 48.26) (xy 57.15 57.15)
+			(xy 57.15 48.26) (xy 57.15 64.77)
 		)
 		(stroke
@@
 	(wire
 		(pts
+			(xy 38.1 64.77) (xy 57.15 64.77)
+		)
+		(stroke
+			(width 0)
+			(type default)
+		)
+	)
+	(wire
+		(pts
 			(xy 176.53 78.74) (xy 194.31 78.74)
 		)
@@
 	(wire
 		(pts
+			(xy 57.15 64.77) (xy 57.15 69.85)
+		)
+		(stroke
+			(width 0)
+			(type default)
+		)
+	)
+	(wire
+		(pts
 			(xy 38.1 88.9) (xy 71.12 88.9)
 		)
@@
 		)
 		(stroke
-			(width 0)
-			(type default)
-		)
-	)
-	(wire
-		(pts
-			(xy 57.15 57.15) (xy 57.15 69.85)
-		)
-		(stroke
